File: PCB/Draft Layouts/draftAccelTemp.sch (EAGLE design)
At the start: 2 parts, among them U1 MMA8452Q

Commit message: Arduino changed
Parts:
- U$1: value ARDUINOUNO -> PRO-MINI-2; device adafruit:ARDUINOUNO -> Arduino-clone:PRO-MINI-2
Connections:
- net N$1: no longer U$1.A5
- net N$2: no longer U$1.A4
- net N$3: no longer U$1.VIN
- net N$4: no longer U$1.GND1
Changed lines of the file:
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@@
 </classes>
 <parts>
-<part name="U$1" library="adafruit" deviceset="ARDUINO" device="UNO"/>
 <part name="U1" library="SparkFun-Sensors" deviceset="MMA8452Q" device=""/>
+<part name="U$1" library="Arduino-clone" deviceset="PRO-MINI-2" device=""/>
 </parts>
 <sheets>
@@
 </plain>
 <instances>
-<instance part="U$1" gate="G$1" x="45.72" y="60.96" smashed="yes"/>
 <instance part="U1" gate="U1" x="132.08" y="104.14" smashed="yes">
 <attribute name="NAME" x="124.46" y="114.554" size="1.778" layer="95" font="vector"/>
 <attribute name="VALUE" x="124.46" y="93.726" size="1.778" layer="96" font="vector" align="top-left"/>
 </instance>
+<instance part="U$1" gate="G$1" x="53.34" y="66.04" smashed="yes"/>
 </instances>
 <busses>
@@
 <net name="N$1" class="0">
 <segment>
-<pinref part="U$1" gate="G$1" pin="A5"/>
 <wire x1="78.74" y1="27.94" x2="154.94" y2="27.94" width="0.1524" layer="91"/>
 <pinref part="U1" gate="U1" pin="SCL"/>
@@
 <net name="N$2" class="0">
 <segment>
-<pinref part="U$1" gate="G$1" pin="A4"/>
 <wire x1="76.2" y1="27.94" x2="76.2" y2="25.4" width="0.1524" layer="91"/>
 <wire x1="76.2" y1="25.4" x2="162.56" y2="25.4" width="0.1524" layer="91"/>
@@
 <wire x1="121.92" y1="111.76" x2="111.76" y2="111.76" width="0.1524" layer="91"/>
 <wire x1="111.76" y1="111.76" x2="111.76" y2="22.86" width="0.1524" layer="91"/>
-<pinref part="U$1" gate="G$1" pin="VIN"/>
 <wire x1="111.76" y1="22.86" x2="60.96" y2="22.86" width="0.1524" layer="91"/>
 <wire x1="60.96" y1="22.86" x2="60.96" y2="27.94" width="0.1524" layer="91"/>
@@
 <net name="N$4" class="0">
 <segment>
-<pinref part="U$1" gate="G$1" pin="GND1"/>
 <wire x1="58.42" y1="27.94" x2="58.42" y2="20.32" width="0.1524" layer="91"/>
 <wire x1="58.42" y1="20.32" x2="116.84" y2="20.32" width="0.1524" layer="91"/>
