File: PCB/MainV2/V2_Layout.brd (EAGLE design)
At the start: 50.1 x 73.7 mm, 48 parts, among them IC1 LM6482, IC2 AD623N, U2 MB85RC256VPF-G-JNERE2

Commit message: Included workarounds in V2 schematic
Parts:
- R3: value 0R -> (none); device rcl:R0603 -> rcl:RTRIM64P
- moved R3 31.1 mm to (12.7, 6.35), turned to 0 degrees
Connections:
- removed net N$6: C3.1, IC2.6
- new net N$17: IC1.3, R3.2
- net +3V3: now also R3.3
- net A0: now also C3.1, IC2.6
- net AGND: now also R7.1; no longer R3.2
- net ECG-REF: now also IC1.1, IC1.2; no longer R3.1
- net GND: now also R3.1; no longer IC1.2, IC1.3, R7.1
Routing:
- net N$6: track 7.95 -> 0.00 mm, vias 1 -> 0
- net A0: track 5.08 -> 13.0 mm, vias 0 -> 1
- net AGND: track 43.2 -> 38.4 mm
