File: PCB/MainV2/V2_Layout.sch (EAGLE design)
At the start: 48 parts, among them IC1 LM6482, IC2 AD623N, U2 MB85RC256VPF-G-JNERE2

Commit message: Included workarounds in V2 schematic
Parts:
- R3: value 0R -> (none); device rcl:R-US_R0603 -> rcl:R-TRIMM64P
Connections:
- removed net N$6: C3.1, IC2.OUT
- new net N$17: IC1A.IN+, R3.S
- net +3V3: now also R3.E
- net A0: now also C3.1, IC2.OUT
- net AGND: now also R7.1; no longer R3.2
- net ECG-REF: now also IC1A.IN-, IC1A.OUT; no longer R3.1
- net GND: now also R3.A; no longer IC1A.IN+, IC1A.IN-, R7.1
Other:
- note added: "Adjustment (temporary)"
- note added: "Adjustment is a workaround to an issue with the critical freqiency of the high-pass filter C3/R7 Pin 6 of the AD623N is connected to A0 in order to determine whether there is saturation of the ECG signal"
- note added: "V2 Notes:"
- note removed: "V1 Notes:"
- moved on the sheet: C10, C11, C5, C8, C9, IC1A, IC1B, R1, R2
